File: water_automation_schematic/garage_schematic.kicad_sch (KiCad schematic)
At the start: 8 parts, among them Q1 BC327, SW1 Button_1, SW2 SW_SPDT, U1 lolin32_lite_V1.00, U2 Relay module

Commit message: edited schematic
Parts:
- added R2, R3: 10k, symbol Device:R
Connections:
- net +3V3: now also R2.1, R3.1
- net at SW2.3 (C), U1.4 (34): now also R2.2
- net at SW1.2, U1.5 (35): now also R3.2
